File: Hardware/S_360_Power_Supply_Adapter.kicad_sch (KiCad schematic)
At the start: 0 parts

Commit message: Finished PCB schematic.
Parts:
- added H1, H2, H3: V+, MountingHole:MountingHole_4.5mm_Pad_Via, symbol Mechanical:MountingHole_Pad
- added H10, H7, H8, H9: MountingHole, MountingHole:MountingHole_4.5mm, symbol Mechanical:MountingHole
- added H4, H5, H6: GND, MountingHole:MountingHole_4.5mm_Pad_Via, symbol Mechanical:MountingHole_Pad
- added J1, J2, J3, J4: PJ-082BH, PJ-082BH:PJ-082BH, symbol PJ-082BH:PJ-082BH
Connections:
- new net GND: H4.1, H5.1, H6.1, J1.2, J1.S1 (Shield), J1.S2 (Shield), J1.S3 (Shield), J1.S4 (Shield), J2.2, J2.S1 (Shield), J2.S2 (Shield), J2.S3 (Shield), J2.S4 (Shield), J3.2, J3.S1 (Shield), J3.S2 (Shield), J3.S3 (Shield), J3.S4 (Shield), J4.2, J4.S1 (Shield), J4.S2 (Shield), J4.S3 (Shield), J4.S4 (Shield)
- new net VDC: H1.1, H2.1, H3.1, J1.1, J2.1, J3.1, J4.1
